File: mm.sch (KiCad schematic (older format))
At the start: 20 parts

Commit message: add info
Connections:
- net 10V: now reaches R4.2, R5.1, SW?.~
- net 50V: now reaches R5.2, R6.1, SW?.~
- net 250V: now reaches R6.2, R7.1, SW?.~
- net ACV_COM: now reaches D1.2 (A), D2.1 (K), SW?.~
- net 0.5mA renamed 0.5mA_DCV_COM
Other:
- note added: "0.15mA"
- note added: "1423 Ohm"
Changed lines of the file:
@@
 	4400 3750 4500 3750
 Text Label 4450 3250 0    50   ~ 0
-0.5mA
+0.5mA_DCV_COM
 Text Label 3900 3150 0    50   ~ 0
 50mA
@@
 Text Notes 2600 4950 1    50   ~ 0
 6.7 Ohm
+Text Notes 3350 5100 0    50   ~ 0
+0.15mA
+Text Label 5950 3650 1    50   ~ 0
+ACV_COM
+Text Label 8050 4850 1    50   ~ 0
+10V
+Text Label 7450 4850 1    50   ~ 0
+50V
+Text Label 6900 4850 1    50   ~ 0
+250V
+Text Notes 5050 3500 0    50   ~ 0
+1423 Ohm
 $EndSCHEMATC

Commit message: add info
Other:
- note added: "let zero adj 1-2 = x Ohm\n\n((2630.7-x)*0.15/(1805.1+x) + 0.15) * 3920 + (2630.7 - x)*0.15 = 1500\n\nx = 425.6 Ohm"
Changed lines of the file:
@@
 Text Notes 5050 3500 0    50   ~ 0
 1423 Ohm
+Text Notes 2100 5900 0    50   ~ 0
+let zero adj 1-2 = x Ohm\n\n((2630.7-x)*0.15/(1805.1+x) + 0.15) * 3920 + (2630.7 - x)*0.15 = 1500\n\nx = 425.6 Ohm
 $EndSCHEMATC
